Commit message: use diffdrive controller

File: catkin_ws/src/rtklm_description/urdf/model.urdf (robot description, URDF)
Before this commit: robot rtklawnmower, 3 links, 2 joints
Links:
- removed link left_wheel_link
- removed link right_wheel_link
- added link base_footprint; visual box size=0.001 0.001 0.001
- added link caster_left_link, mass 0.5; collision sphere radius=0.025; visual sphere radius=0.025
- added link caster_right_link, mass 0.5; collision sphere radius=0.025; visual sphere radius=0.025
- added link left_wheel, mass 0.5; collision cylinder length=0.08 radius=0.06; visual cylinder length=0.08 radius=0.06
- added link right_wheel, mass 0.5; collision cylinder length=0.08 radius=0.06; visual cylinder length=0.08 radius=0.06
- link base_link: mass 10 -> 4; geometry collision box size=0.40 0.25 0.10; visual box size=0.4 0.25 0.1
Joints:
- removed joint base_to_left_wheel_joint
- removed joint base_to_right_wheel_joint
- added joint base_footprint_joint: type fixed, parent base_footprint, child base_link, origin xyz=0 0 0.06 rpy=0 0 0
- added joint caster_left_joint: type fixed, parent base_link, child caster_left_link, origin xyz=0.3 -0.1 0.01 rpy=-${pi/2} 0 0
- added joint caster_right_joint: type fixed, parent base_link, child caster_right_link, origin xyz=0.3 0.1 0.01 rpy=-${pi/2} 0 0
- added joint left_wheel_joint: type continuous, parent base_link, child left_wheel, origin xyz=0.0 -0.08 0.0 rpy=0 0 0, axis 0 1 0, limit effort=100 velocity=100
- added joint right_wheel_joint: type continuous, parent base_link, child right_wheel, origin xyz=0.0 0.08 0.0 rpy=0 0 0, axis 0 1 0, limit effort=100 velocity=100

Commit message: Optimized caster wheels

File: catkin_ws/src/rtklm_description/urdf/model.urdf (robot description, URDF)
Before this commit: robot rtklawnmower, 6 links, 5 joints
Links:
- removed link caster_left_link
- removed link caster_right_link
- added link left_caster, mass 0.1; collision sphere radius=0.04; visual sphere radius=0.04
- added link right_caster, mass 0.1; collision sphere radius=0.04; visual sphere radius=0.04
Joints:
- joint caster_left_joint: child caster_left_link -> left_caster; origin xyz=0.3 -0.1 0.01 rpy=-${pi/2} 0 0 -> xyz=0.25 -0.1 -0.01 rpy=0 0 0
- joint caster_right_joint: child caster_right_link -> right_caster; origin xyz=0.3 0.1 0.01 rpy=-${pi/2} 0 0 -> xyz=0.25 0.1 -0.01 rpy=0 0 0

Commit message: Simplify by using a little xacro

File: catkin_ws/src/rtklm_description/urdf/model.urdf (robot description, URDF)
Before this commit: robot rtklawnmower, 6 links, 5 joints
Links:
- link base_link: mass 4 -> None; geometry collision box size=${chassis_l} ${chassis_w} ${chassis_h}; visual box size=${chassis_l} ${chassis_w} ${chassis_h}
- link left_caster: mass 0.1 -> None; geometry collision sphere radius=${caster_r}; visual sphere radius=${caster_r}
- link left_wheel: mass 0.5 -> None; geometry collision cylinder length=${wheel_l} radius=${wheel_r}; visual cylinder length=${wheel_l} radius=${wheel_r}
- link right_caster: mass 0.1 -> None; geometry collision sphere radius=${caster_r}; visual sphere radius=${caster_r}
- link right_wheel: mass 0.5 -> None; geometry collision cylinder length=${wheel_l} radius=${wheel_r}; visual cylinder length=${wheel_l} radius=${wheel_r}
Joints:
- joint left_wheel_joint: limit effort=100 velocity=100 -> (none)
- joint right_wheel_joint: limit effort=100 velocity=100 -> (none)
