Commit message: Add state publisher for transforms, prepare localization

File: catkin_ws/src/rtklm_description/urdf/imu.xacro (robot description, xacro)
@@ -1,8 +1,8 @@
 <?xml version="1.0"?>
 <robot xmlns:xacro="http://www.ros.org/wiki/xacro" name="rtklawnmower">
-  <xacro:macro name="imu" params="length width height mass offset">
+  <xacro:macro name="imu" params="length width height mass joint_offset">
     <link name="imu_link">
         <visual>
-            <origin xyz="${offset}" rpy="0 0 0"/>
+            <origin xyz="0 0 0" rpy="0 0 0"/>
             <geometry>
                 <box size="${length} ${width} ${height}"/>
@@ -10,5 +10,5 @@
         </visual>
         <collision>
-            <origin xyz="${offset}" rpy="0 0 0"/>
+            <origin xyz="0 0 0" rpy="0 0 0"/>
             <geometry>
                 <box size="${length} ${width} ${height}"/>
@@ -16,5 +16,5 @@
         </collision>
         <inertial>
-            <origin xyz="${offset}" rpy="0 0 0"/>
+            <origin xyz="0 0 0" rpy="0 0 0"/>
             <mass value="${mass}"/>
             <inertia ixx="${(1/12) * mass * (width*width + height*height)}" ixy="0.0" ixz="0.0"
@@ -23,4 +23,9 @@
         </inertial>
     </link>
+    <joint name="imu_joint" type="fixed">
+        <origin xyz="${joint_offset}" rpy="0 0 0"/>
+        <parent link="base_link"/>
+        <child link="imu_link"/>
+    </joint>
     <gazebo reference="imu_link">
         <mu1>0.3</mu1>

File: catkin_ws/src/rtklm_description/urdf/main.xacro (robot description, xacro)
@@ -13,5 +13,5 @@
     <!-- IMU -->
     <xacro:include filename="$(find rtklm_description)/urdf/imu.xacro" />
-    <xacro:imu length="0.02" width="0.03" height="0.01" mass="0.01" offset="0.00 0.00 0.30" -->
+    <xacro:imu length="0.03" width="0.02" height="0.01" mass="0.01" joint_offset="0.00 0.00 0.08" />
     <!-- differential drive wheels -->
     <xacro:include filename="$(find rtklm_description)/urdf/wheel.xacro" />
