Commit message: Limit wheel joint efforts to they don't implode to origin and adjust Gazebo parameters so rover will not slip

File: catkin_ws/src/rtklm_description/urdf/casterwheel.xacro (robot description, xacro)
@@ -28,4 +28,9 @@
         <origin xyz="${joint_offset}" rpy="0 0 0"/>
     </joint>
+    <gazebo reference="${prefix}_casterwheel">
+        <mu1>0.0</mu1>
+        <mu2>0.0</mu2>
+        <material>Gazebo/FlatBlack</material>
+    </gazebo>
   </xacro:macro>
 </robot>

File: catkin_ws/src/rtklm_description/urdf/main.xacro (robot description, xacro)
@@ -1,31 +1,22 @@
 <?xml version="1.0"?>
 <robot xmlns:xacro="http://www.ros.org/wiki/xacro" name="rtklawnmower">
+    <xacro:include filename="$(find rtklm_description)/urdf/chassis.xacro" />
     <xacro:include filename="$(find rtklm_description)/urdf/wheel.xacro" />
     <xacro:include filename="$(find rtklm_description)/urdf/casterwheel.xacro" />
-    <link name="base_link">
-        <visual>
-            <origin xyz="0.13 0 0.11" rpy="0 0 0"/>
-            <geometry>
-                <box size="0.40 0.25 0.10"/>
-            </geometry>
-        </visual>
-        <collision>
-            <origin xyz="0.13 0 0.11" rpy="0 0 0"/>
-            <geometry>
-                <box size="0.40 0.25 0.10"/>
-            </geometry>
-        </collision>
-        <inertial>
-            <origin xyz="0.13 0 0.11" rpy="0 0 0"/>
-            <mass value="4"/>
-            <inertia ixx="${(1/12) * 4 * (0.25*0.25 + 0.10*0.10)}" ixy="0.0" ixz="0.0"
-                     iyy="${(1/12) * 4 * (0.40*0.40 + 0.10*0.10)}" iyz="0.0"
-                     izz="${(1/12) * 4 * (0.40*0.40 + 0.25*0.25)}" />
-        </inertial>
-    </link>
-    <xacro:wheel prefix="right" radius="0.06" length="0.08" mass="0.5" joint_offset="0 -0.1 0" />
-    <xacro:wheel prefix="left"  radius="0.06" length="0.08" mass="0.5" joint_offset="0  0.1 0" />
-    <xacro:casterwheel prefix="right" radius="0.04" mass="0.1" joint_offset="0.25 -0.1 -0.02" />
-    <xacro:casterwheel prefix="left"  radius="0.04" mass="0.1" joint_offset="0.25  0.1 -0.02" />
+    <!-- base_footprint is a fictitious link(frame) that is on the ground right below base_link origin -->
+    <link name="base_footprint" />
+    <joint name="base_footprint_joint" type="fixed">
+      <parent link="base_footprint"/>
+      <child link="base_link" />
+      <origin xyz="0 0 0.06" rpy="0 0 0" />
+    </joint>
+    <!-- chassis is in base_link-->
+    <xacro:chassis length="0.40" width="0.25" height="0.10" mass="4" offset="0.13 0.00 0.11" />
+    <!-- differential drive wheels -->
+    <xacro:wheel prefix="right" radius="0.06" length="0.08" mass="0.5" joint_offset="0.0 -0.1 0.0" />
+    <xacro:wheel prefix="left"  radius="0.06" length="0.08" mass="0.5" joint_offset="0.0  0.1 0.0" />
+    <!-- caster wheels -->
+    <xacro:casterwheel prefix="right" radius="0.04" mass="0.1" joint_offset="0.25 -0.10 -0.02" />
+    <xacro:casterwheel prefix="left"  radius="0.04" mass="0.1" joint_offset="0.25  0.10 -0.02" />
     <gazebo>
         <plugin name="gazebo_ros_control" filename="libgazebo_ros_control.so">

File: catkin_ws/src/rtklm_description/urdf/wheel.xacro (robot description, xacro)
@@ -28,4 +28,5 @@
         <child link="${prefix}_wheel"/>
         <origin xyz="${joint_offset}" rpy="0 0 0"/>
+        <limit effort="100" velocity="100"/>
     </joint>
     <transmission name="${prefix}_wheel_transmission">
@@ -33,4 +34,5 @@
         <actuator name="${prefix}_wheel_motor">
             <mechanicalReduction>1</mechanicalReduction>
+            <hardwareInterface>hardware_interface/VelocityJointInterface</hardwareInterface>
         </actuator>
         <joint name="${prefix}_wheel_joint">
@@ -38,4 +40,13 @@
         </joint>
     </transmission>
+    <gazebo reference="${prefix}_wheel">
+      <mu1 value="1.0"/>
+      <mu2 value="1.0"/>
+      <kp  value="10000000.0" />
+      <kd>100.0</kd>
+      <minDepth>0.001</minDepth>
+      <maxVel>0.1</maxVel>
+      <material>Gazebo/FlatBlack</material>
+    </gazebo>
   </xacro:macro>
 </robot>

Commit message: Remove gazebo config, adjust to 10Hz Arduino node

File: catkin_ws/src/rtklm_description/urdf/casterwheel.xacro (robot description, xacro)
@@ -28,9 +28,4 @@
         <origin xyz="${joint_offset}" rpy="0 0 0"/>
     </joint>
-    <gazebo reference="${prefix}_casterwheel">
-        <mu1>0.0</mu1>
-        <mu2>0.0</mu2>
-        <material>Gazebo/FlatBlack</material>
-    </gazebo>
   </xacro:macro>
 </robot>

File: catkin_ws/src/rtklm_description/urdf/chassis.xacro (robot description, xacro)
@@ -23,9 +23,4 @@
         </inertial>
     </link>
-    <gazebo reference="base_link">
-        <mu1>0.3</mu1>
-        <mu2>0.3</mu2>
-        <material>Gazebo/Green</material>
-    </gazebo>
   </xacro:macro>
 </robot>

File: catkin_ws/src/rtklm_description/urdf/imu.xacro (robot description, xacro)
@@ -28,9 +28,4 @@
         <child link="imu_link"/>
     </joint>
-    <gazebo reference="imu_link">
-        <mu1>0.3</mu1>
-        <mu2>0.3</mu2>
-        <material>Gazebo/Green</material>
-    </gazebo>
   </xacro:macro>
 </robot>

File: catkin_ws/src/rtklm_description/urdf/main.xacro (robot description, xacro)
@@ -22,8 +22,3 @@
     <xacro:casterwheel prefix="right" radius="0.04" mass="0.1" joint_offset="0.25 -0.10 -0.02" />
     <xacro:casterwheel prefix="left"  radius="0.04" mass="0.1" joint_offset="0.25  0.10 -0.02" />
-    <gazebo>
-        <plugin name="gazebo_ros_control" filename="libgazebo_ros_control.so">
-            <robotNamespace>/</robotNamespace>
-        </plugin>
-    </gazebo>
 </robot>

File: catkin_ws/src/rtklm_description/urdf/wheel.xacro (robot description, xacro)
@@ -40,13 +40,4 @@
     </transmission>
 -->
-    <gazebo reference="${prefix}_wheel">
-      <mu1 value="1.0"/>
-      <mu2 value="1.0"/>
-      <kp  value="10000000.0" />
-      <kd>100.0</kd>
-      <minDepth>0.001</minDepth>
-      <maxVel>0.1</maxVel>
-      <material>Gazebo/FlatBlack</material>
-    </gazebo>
   </xacro:macro>
 </robot>
